Commit message: add new world

File: src/world_pkg/urdf/form.urdf (robot description, URDF)
Before this commit: robot cubs, 1 links, 0 joints
Links:
- removed link cub
- added link form, mass 0.2; collision mesh filename=package://world_pkg/meshes/form.dae scale=0.001 0.001 0.001; visual mesh filename=package://world_pkg/meshes/form.dae scale=0.001 0.001 0.001
